Commit message: added joint state publisher

File: ribot_description/urdf/robot.urdf.xacro (robot description, xacro)
@@ -85,8 +85,12 @@
     </link>
     <!-- tripod to tripod plate-->
-    <joint name="tripod_to_tripod_plate" type="fixed">
+    <joint name="tripod_to_tripod_plate" type="revolute">
         <parent link="tripod" />
         <child link="tripod_plate" />
         <origin xyz=".01 .03 1.65" rpy="0 0.314 0" />
+        <!-- <calibration rising="0.0"/> -->
+        <!-- <dynamics damping="0.0" friction="0.0"/> -->
+        <limit effort="30" velocity="1.0" lower="-2.2" upper="0.7" />
+        <!-- <safety_controller k_velocity="10" k_position="15" soft_lower_limit="-2.0" soft_upper_limit="0.5" /> -->
     </joint>
     <!-- Tripod left support-->

Commit message: tidying up

File: ribot_description/urdf/robot.urdf.xacro (robot description, xacro)
@@ -17,5 +17,5 @@
     <!-- Left IMU -->
     <xacro:imu parent="tripod_left_support" prefix="imu" color_gazebo="Red">
-        <origin xyz="0.015 0 0.012" rpy="0 0 0" />
+        <origin xyz="0.015 0 0.02" rpy="0 0 0" />
         <color_rgb_rviz>
             <material name="red">

Commit message: reworking the system
addidng gazebo controllers so the system is properly created and
functional; the goal is to be able to move the robot with 6 DOF - for
that, the gazebo joint controllers need to be set up - currently working
on that

File: ribot_description/urdf/robot.urdf.xacro (robot description, xacro)
@@ -1,14 +1,20 @@
 <?xml version="1.0"?>
-<robot name="robot" xmlns:xacro="http://ros.org/wiki/xacro">
+<robot name="ribot" xmlns:xacro="http://ros.org/wiki/xacro">
     <!-- ribot is a simple robotic system containing one rgb camera and an imu on top of a tripop.  -->
     <!-- Define  properties -->
     <xacro:property name="M_PI" value="3.1415926535897931" />
     <material name="Orange">
-        <color rgba="1.0 0.4 0.0 1.0" />
+        <color rgba="1.0 0.4 0.0 1.0"/>
     </material>
     <!-- Colors -->
     <material name="tripod_color">
-        <color rgba="0.21 0.21 .21 1" />
+        <color rgba="0.21 0.21 .21 1"/>
     </material>
+    <xacro:macro name="default_inertial">
+        <inertial>
+            <mass value="1"/>
+            <inertia ixx="1.0" ixy="0.0" ixz="0.0" iyy="1.0" iyz="0.0" izz="1.0" />
+        </inertial>
+    </xacro:macro>
     <!-- Includes -->
     <xacro:include filename="$(find ribot_description)/urdf/robot.gazebo.xacro" />
@@ -17,7 +23,66 @@
     <!-- World link -->
     <link name="world"/>
-    <joint name="world_to_plate" type="fixed">
+    <!-- Simulation of a 6DOF ("floating") joint through the creation of 6 joints -->
+    <joint name="world_to_d_prismatic_x" type="prismatic">
         <parent link="world"/>
+        <child link="d_prismatic_x"/>
+        <axis xyz="1 0 0"/>
+        <limit effort="1000.0" lower="-10" upper="10" velocity="0.5"/>
+        <origin rpy="0 0 0" xyz="0 0 0"/>
+    </joint>
+    <link name="d_prismatic_x">
+        <xacro:default_inertial />
+    </link>
+    <joint name="d_prismatic_x_to_d_prismatic_y" type="prismatic">
+        <parent link="d_prismatic_x"/>
+        <child link="d_prismatic_y"/>
+        <axis xyz="0 1 0"/>
+        <limit effort="1000.0" lower="-10" upper="10" velocity="0.5"/>
+        <origin rpy="0 0 0" xyz="0 0 0"/>
+    </joint>
+    <link name="d_prismatic_y">
+        <xacro:default_inertial />
+    </link>
+    <joint name="d_prismatic_y_to_d_prismatic_z" type="prismatic">
+        <parent link="d_prismatic_y"/>
+        <child link="d_prismatic_z"/>
+        <axis xyz="0 0 1"/>
+        <limit effort="1000.0" lower="-10" upper="10" velocity="0.5"/>
+        <origin rpy="0 0 0" xyz="0 0 0"/>
+    </joint>
+    <link name="d_prismatic_z">
+        <xacro:default_inertial />
+    </link>
+    <joint name="d_prismatic_z_to_d_revolute_x" type="continuous">
+        <parent link="d_prismatic_z"/>
+        <child link="d_revolute_x"/>
+        <axis xyz="1 0 0"/>
+        <origin xyz="0 0 0"/>
+    </joint>
+    <link name="d_revolute_x">
+        <xacro:default_inertial />
+    </link>
+    <joint name="d_revolute_x_to_d_revolute_y" type="continuous">
+        <parent link="d_revolute_x"/>
+        <child link="d_revolute_y"/>
+        <axis xyz="0 1 0"/>
+        <origin xyz="0 0 0"/>
+    </joint>
+    <link name="d_revolute_y">
+        <xacro:default_inertial />
+    </link>
+    <joint name="d_revolute_y_to_d_revolute_z" type="continuous">
+        <parent link="d_revolute_y"/>
+        <child link="d_revolute_z"/>
+        <axis xyz="0 0 1"/>
+        <origin xyz="0 0 0"/>
+    </joint>
+    <link name="d_revolute_z">
+        <xacro:default_inertial />
+    </link>
+    <joint name="d_revolute_z_to_plate" type="fixed">
+        <parent link="d_revolute_z"/>
         <child link="plate"/>
+        <origin xyz="0 0 0"/>
     </joint>
     <link name="plate">
@@ -35,12 +100,8 @@
             </geometry>
         </collision>
-        <inertial>
-            <mass value="1.0" />
-            <origin xyz="0 0 0" rpy="0 0 0" />
-            <inertia ixx="1" ixy="0" ixz="0" iyy="1" iyz="0" izz="1" />
-        </inertial>
-        <gazebo>
+        <xacro:default_inertial />
+        <!-- <gazebo>
             <gravity>0</gravity>
-        </gazebo>
+        </gazebo> -->
     </link>
     <!-- Tripod left support-->
@@ -79,16 +140,18 @@
         </color_rgb_rviz>
     </xacro:rgb_camera>
-    <!-- Gazebo Plugin that publishes the GT IMU TF to a specified topic -->
+    <!-- Gazebo Joint Control Plugins and Transmissions -->
     <gazebo>
-        <plugin name="p3d_base_controller" filename="libgazebo_ros_p3d.so">
-        <alwaysOn>true</alwaysOn>
-        <updateRate>200.0</updateRate>
-        <bodyName>imu_link</bodyName>
-        <topicName>ground_truth/imu_tf</topicName>
-        <gaussianNoise>0.00</gaussianNoise>
-        <frameName>world</frameName>
-        <xyzOffsets>0 0 0</xyzOffsets>
-        <rpyOffsets>0 0 0</rpyOffsets>
+        <plugin name="gazebo_ros_control" filename="libgazebo_ros_control.so">
+            <robotNamespace>/</robotNamespace>
         </plugin>
     </gazebo>
+    <transmission name="world_to_d_prismatic_x_trans">
+        <type>transmission_interface/SimpleTransmission</type>
+        <actuator name="motor1">
+            <mechanicalReduction>1</mechanicalReduction>
+        </actuator>
+        <joint name="world_to_d_prismatic_x">
+            <hardwareInterface>hardware_interface/PositionJointInterface</hardwareInterface>
+        </joint>
+    </transmission>
 </robot>

Commit message: Simple test for gazebo Fixes #1

File: ribot_description/urdf/robot.urdf.xacro (robot description, xacro)
@@ -22,67 +22,11 @@
     <xacro:include filename="$(find ribot_description)/urdf/imu.urdf.xacro"/>
     <!-- World link -->
-    <link name="world"/>
-    <!-- Simulation of a 6DOF ("floating") joint through the creation of 6 joints -->
-    <joint name="world_to_d_prismatic_x" type="prismatic">
-        <parent link="world"/>
-        <child link="d_prismatic_x"/>
-        <axis xyz="1 0 0"/>
-        <limit effort="1000.0" lower="-10" upper="10" velocity="0.5"/>
-        <origin rpy="0 0 0" xyz="0 0 0"/>
-    </joint>
-    <link name="d_prismatic_x">
-        <xacro:default_inertial />
+    <!-- <link name="world"/> -->
+    <link name="base_link">
     </link>
-    <joint name="d_prismatic_x_to_d_prismatic_y" type="prismatic">
-        <parent link="d_prismatic_x"/>
-        <child link="d_prismatic_y"/>
-        <axis xyz="0 1 0"/>
-        <limit effort="1000.0" lower="-10" upper="10" velocity="0.5"/>
-        <origin rpy="0 0 0" xyz="0 0 0"/>
-    </joint>
-    <link name="d_prismatic_y">
-        <xacro:default_inertial />
-    </link>
-    <joint name="d_prismatic_y_to_d_prismatic_z" type="prismatic">
-        <parent link="d_prismatic_y"/>
-        <child link="d_prismatic_z"/>
-        <axis xyz="0 0 1"/>
-        <limit effort="1000.0" lower="-10" upper="10" velocity="0.5"/>
-        <origin rpy="0 0 0" xyz="0 0 0"/>
-    </joint>
-    <link name="d_prismatic_z">
-        <xacro:default_inertial />
-    </link>
-    <joint name="d_prismatic_z_to_d_revolute_x" type="continuous">
-        <parent link="d_prismatic_z"/>
-        <child link="d_revolute_x"/>
-        <axis xyz="1 0 0"/>
-        <origin xyz="0 0 0"/>
-    </joint>
-    <link name="d_revolute_x">
-        <xacro:default_inertial />
-    </link>
-    <joint name="d_revolute_x_to_d_revolute_y" type="continuous">
-        <parent link="d_revolute_x"/>
-        <child link="d_revolute_y"/>
-        <axis xyz="0 1 0"/>
-        <origin xyz="0 0 0"/>
-    </joint>
-    <link name="d_revolute_y">
-        <xacro:default_inertial />
-    </link>
-    <joint name="d_revolute_y_to_d_revolute_z" type="continuous">
-        <parent link="d_revolute_y"/>
-        <child link="d_revolute_z"/>
-        <axis xyz="0 0 1"/>
-        <origin xyz="0 0 0"/>
-    </joint>
-    <link name="d_revolute_z">
-        <xacro:default_inertial />
-    </link>
-    <joint name="d_revolute_z_to_plate" type="fixed">
-        <parent link="d_revolute_z"/>
-        <child link="plate"/>
-        <origin xyz="0 0 0"/>
+    <joint name="base_link_to_plate" type="fixed">
+      <origin xyz="0 0 0" rpy="0 0 0"/>
+      <parent link="base_link"/>
+      <child link="plate"/>
     </joint>
     <link name="plate">
@@ -101,57 +45,14 @@
         </collision>
         <xacro:default_inertial />
-        <!-- <gazebo>
+        <gazebo>
             <gravity>0</gravity>
-        </gazebo> -->
+        </gazebo>
     </link>
-    <!-- Tripod left support-->
-    <link name="left_support" />
-    <!-- tripod plate to tripod left support -->
-    <joint name="plate_to_left_support" type="fixed">
-        <parent link="plate" />
-        <child link="left_support" />
-        <origin xyz="0 0.18 0.0075" rpy="0 0 0" />
+    <link name="imu">
+    </link>
+    <joint name="plate_to_imu" type="fixed">
+      <origin xyz="0 0.1 -0.305" rpy="0 0 0"/>
+      <parent link="plate"/>
+      <child link="imu"/>
     </joint>
-    <!-- Tripod right support-->
-    <link name="right_support" />
-    <!-- tripod plate to tripod right support -->
-    <joint name="plate_to_right_support" type="fixed">
-        <parent link="plate" />
-        <child link="right_support" />
-        <origin xyz="0 -0.18 0.0075" rpy="0 0 0" />
-    </joint>
-    <!-- SENSORS -->
-    <!-- Left IMU -->
-    <xacro:imu parent="left_support" prefix="imu" color_gazebo="Red">
-        <origin xyz="0.015 0 0.02" rpy="0 0 0" />
-        <color_rgb_rviz>
-            <material name="red">
-                <color rgba="0.9 0 0 1" />
-            </material>
-        </color_rgb_rviz>
-    </xacro:imu>
-    <!-- Right Camera -->
-    <xacro:rgb_camera parent="right_support" prefix="rgb_right" color_gazebo="Green">
-        <origin xyz="0.015 0 0.012" rpy="0 0 0" />
-        <color_rgb_rviz>
-            <material name="green">
-                <color rgba="0 0.9 0 1" />
-            </material>
-        </color_rgb_rviz>
-    </xacro:rgb_camera>
-    <!-- Gazebo Joint Control Plugins and Transmissions -->
-    <gazebo>
-        <plugin name="gazebo_ros_control" filename="libgazebo_ros_control.so">
-            <robotNamespace>/</robotNamespace>
-        </plugin>
-    </gazebo>
-    <transmission name="world_to_d_prismatic_x_trans">
-        <type>transmission_interface/SimpleTransmission</type>
-        <actuator name="motor1">
-            <mechanicalReduction>1</mechanicalReduction>
-        </actuator>
-        <joint name="world_to_d_prismatic_x">
-            <hardwareInterface>hardware_interface/PositionJointInterface</hardwareInterface>
-        </joint>
-    </transmission>
 </robot>
