Commit message: fix: prismatic joint now can be controlled
adding an explicit lower and upper limit to the prismatic joint
position fixed the issue; the default values are 0 and as such, the
joint wouldn't move

File: ribot_description/urdf/robot2.urdf.xacro (robot description, xacro)
@@ -22,8 +22,19 @@
     </link>
     <!-- Joint connecting the base link to the second link -->
-    <joint name="base_link_to_revolute_x" type="continuous">
+    <joint name="base_link_to_prismatic_x" type="prismatic">
         <origin xyz="0 0 0" rpy="0 0 0"/>
         <axis xyz="1 0 0"/>
         <parent link="base_link"/>
+        <child link="prismatic_x"/>
+        <limit effort="30" velocity="1.0" lower="-10000" upper="10000"/>
+    </joint>
+    <link name="prismatic_x">
+        <origin xyz="0 0 0" rpy="0 0 0"/>
+        <xacro:default_inertial/>
+    </link>
+    <joint name="prismatic_x_to_revolute_x" type="continuous">
+        <origin xyz="0 0 0" rpy="0 0 0"/>
+        <axis xyz="1 0 0"/>
+        <parent link="prismatic_x"/>
         <child link="revolute_x"/>
         <limit effort="30" velocity="1.0"/>
@@ -55,18 +66,7 @@
         <xacro:default_inertial/>
     </link>
-    <joint name="revolute_z_to_prismatic_x" type="prismatic">
-        <origin xyz="0 0 0" rpy="0 0 0"/>
-        <axis xyz="1 0 0"/>
+    <joint name="revolute_z_to_plate" type="fixed">
+        <origin xyz="0 0 0.0075" rpy="0 0 0"/>
         <parent link="revolute_z"/>
-        <child link="prismatic_x"/>
-        <limit effort="3000" velocity="30.0"/>
-    </joint>
-    <link name="prismatic_x">
-        <origin xyz="0 0 0" rpy="0 0 0"/>
-        <xacro:default_inertial/>
-    </link>
-    <joint name="prismatic_x_to_plate" type="fixed">
-        <origin xyz="0 0 0.0075" rpy="0 0 0"/>
-        <parent link="prismatic_x"/>
         <child link="plate"/>
     </joint>
@@ -93,10 +93,19 @@
     </gazebo>
     <!-- Transmissions -->
-    <transmission name="base_link_to_revolute_x_trans">
+    <transmission name="base_link_to_prismatic_x_trans">
         <type>transmission_interface/SimpleTransmission</type>
         <actuator name="motor1">
             <mechanicalReduction>1</mechanicalReduction>
         </actuator>
-        <joint name="base_link_to_revolute_x">
+        <joint name="base_link_to_prismatic_x">
+            <hardwareInterface>hardware_interface/PositionJointInterface</hardwareInterface>
+        </joint>
+    </transmission>
+    <transmission name="prismatic_x_to_revolute_x_trans">
+        <type>transmission_interface/SimpleTransmission</type>
+        <actuator name="motor2">
+            <mechanicalReduction>1</mechanicalReduction>
+        </actuator>
+        <joint name="prismatic_x_to_revolute_x">
             <hardwareInterface>hardware_interface/PositionJointInterface</hardwareInterface>
         </joint>
@@ -104,5 +113,5 @@
     <transmission name="revolute_x_to_revolute_y_trans">
         <type>transmission_interface/SimpleTransmission</type>
-        <actuator name="motor2">
+        <actuator name="motor3">
             <mechanicalReduction>1</mechanicalReduction>
         </actuator>
@@ -113,5 +122,5 @@
     <transmission name="revolute_y_to_revolute_z_trans">
         <type>transmission_interface/SimpleTransmission</type>
-        <actuator name="motor3">
+        <actuator name="motor4">
             <mechanicalReduction>1</mechanicalReduction>
         </actuator>
@@ -120,12 +129,3 @@
         </joint>
     </transmission>
-    <transmission name="revolute_z_to_prismatic_x_trans">
-        <type>transmission_interface/SimpleTransmission</type>
-        <actuator name="motor4">
-            <mechanicalReduction>1</mechanicalReduction>
-        </actuator>
-        <joint name="revolute_z_to_prismatic_x">
-            <hardwareInterface>hardware_interface/PositionJointInterface</hardwareInterface>
-        </joint>
-    </transmission>
 </robot>

Commit message: fix: added a prismatic Y joint and its control

File: ribot_description/urdf/robot2.urdf.xacro (robot description, xacro)
@@ -33,8 +33,19 @@
         <xacro:default_inertial/>
     </link>
-    <joint name="prismatic_x_to_revolute_x" type="continuous">
+    <joint name="prismatic_x_to_prismatic_y" type="prismatic">
+        <origin xyz="0 0 0" rpy="0 0 0"/>
+        <axis xyz="0 1 0"/>
+        <parent link="prismatic_x"/>
+        <child link="prismatic_y"/>
+        <limit effort="30" velocity="1.0" lower="-10000" upper="10000"/>
+    </joint>
+    <link name="prismatic_y">
+        <origin xyz="0 0 0" rpy="0 0 0"/>
+        <xacro:default_inertial/>
+    </link>
+    <joint name="prismatic_y_to_revolute_x" type="continuous">
         <origin xyz="0 0 0" rpy="0 0 0"/>
         <axis xyz="1 0 0"/>
-        <parent link="prismatic_x"/>
+        <parent link="prismatic_y"/>
         <child link="revolute_x"/>
         <limit effort="30" velocity="1.0"/>
@@ -102,10 +113,19 @@
         </joint>
     </transmission>
-    <transmission name="prismatic_x_to_revolute_x_trans">
+    <transmission name="prismatic_x_to_prismatic_y_trans">
         <type>transmission_interface/SimpleTransmission</type>
         <actuator name="motor2">
             <mechanicalReduction>1</mechanicalReduction>
         </actuator>
-        <joint name="prismatic_x_to_revolute_x">
+        <joint name="prismatic_x_to_prismatic_y">
+            <hardwareInterface>hardware_interface/PositionJointInterface</hardwareInterface>
+        </joint>
+    </transmission>
+    <transmission name="prismatic_y_to_revolute_x_trans">
+        <type>transmission_interface/SimpleTransmission</type>
+        <actuator name="motor3">
+            <mechanicalReduction>1</mechanicalReduction>
+        </actuator>
+        <joint name="prismatic_y_to_revolute_x">
             <hardwareInterface>hardware_interface/PositionJointInterface</hardwareInterface>
         </joint>
@@ -113,5 +133,5 @@
     <transmission name="revolute_x_to_revolute_y_trans">
         <type>transmission_interface/SimpleTransmission</type>
-        <actuator name="motor3">
+        <actuator name="motor4">
             <mechanicalReduction>1</mechanicalReduction>
         </actuator>
@@ -122,5 +142,5 @@
     <transmission name="revolute_y_to_revolute_z_trans">
         <type>transmission_interface/SimpleTransmission</type>
-        <actuator name="motor4">
+        <actuator name="motor5">
             <mechanicalReduction>1</mechanicalReduction>
         </actuator>

Commit message: fix: added prismatic z joint and its control
now the robot features ROS control for all of the 6 DOF of movement;

File: ribot_description/urdf/robot2.urdf.xacro (robot description, xacro)
@@ -44,8 +44,19 @@
         <xacro:default_inertial/>
     </link>
-    <joint name="prismatic_y_to_revolute_x" type="continuous">
+    <joint name="prismatic_y_to_prismatic_z" type="prismatic">
+        <origin xyz="0 0 0" rpy="0 0 0"/>
+        <axis xyz="0 0 1"/>
+        <parent link="prismatic_y"/>
+        <child link="prismatic_z"/>
+        <limit effort="30" velocity="1.0" lower="-10000" upper="10000"/>
+    </joint>
+    <link name="prismatic_z">
+        <origin xyz="0 0 0" rpy="0 0 0"/>
+        <xacro:default_inertial/>
+    </link>
+    <joint name="prismatic_z_to_revolute_x" type="continuous">
         <origin xyz="0 0 0" rpy="0 0 0"/>
         <axis xyz="1 0 0"/>
-        <parent link="prismatic_y"/>
+        <parent link="prismatic_z"/>
         <child link="revolute_x"/>
         <limit effort="30" velocity="1.0"/>
@@ -122,10 +133,19 @@
         </joint>
     </transmission>
-    <transmission name="prismatic_y_to_revolute_x_trans">
+    <transmission name="prismatic_y_to_prismatic_z_trans">
         <type>transmission_interface/SimpleTransmission</type>
         <actuator name="motor3">
             <mechanicalReduction>1</mechanicalReduction>
         </actuator>
-        <joint name="prismatic_y_to_revolute_x">
+        <joint name="prismatic_y_to_prismatic_z">
+            <hardwareInterface>hardware_interface/PositionJointInterface</hardwareInterface>
+        </joint>
+    </transmission>
+    <transmission name="prismatic_z_to_revolute_x_trans">
+        <type>transmission_interface/SimpleTransmission</type>
+        <actuator name="motor4">
+            <mechanicalReduction>1</mechanicalReduction>
+        </actuator>
+        <joint name="prismatic_z_to_revolute_x">
             <hardwareInterface>hardware_interface/PositionJointInterface</hardwareInterface>
         </joint>
@@ -133,5 +153,5 @@
     <transmission name="revolute_x_to_revolute_y_trans">
         <type>transmission_interface/SimpleTransmission</type>
-        <actuator name="motor4">
+        <actuator name="motor5">
             <mechanicalReduction>1</mechanicalReduction>
         </actuator>
@@ -142,5 +162,5 @@
     <transmission name="revolute_y_to_revolute_z_trans">
         <type>transmission_interface/SimpleTransmission</type>
-        <actuator name="motor5">
+        <actuator name="motor6">
             <mechanicalReduction>1</mechanicalReduction>
         </actuator>
