Commit message: removed imu gazebo plugin from system

File: ribot_description/urdf/imu.urdf.xacro (robot description, xacro)
@@ -37,72 +37,24 @@
 		</link>
 		<!-- IMU sensor-->
-		<gazebo reference="${prefix}_link">
-			<sensor type="imu" name="imu_sensor">
-                <always_on>1</always_on>
-                <update_rate>1</update_rate>
-                <visualize>true</visualize>
-                <topic>imu</topic>
-				<plugin name="${prefix}_plugin" filename="libgazebo_ros_imu_sensor.so">
-					<topicName>imu_data</topicName>
-                    <!-- <bodyName>${prefix}_link</bodyName> -->
-                    <updateRateHz>10.0</updateRateHz>
-                    <frameName>${prefix}_link</frameName>
-                </plugin>
-                <!-- <imu>
-                <angular_velocity>
-                    <x>
-                    <noise type="gaussian">
-                        <mean>0.0</mean>
-                        <stddev>2e-4</stddev>
-                        <bias_mean>0.0000075</bias_mean>
-                        <bias_stddev>0.0000008</bias_stddev>
-                    </noise>
-                    </x>
-                    <y>
-                    <noise type="gaussian">
-                        <mean>0.0</mean>
-                        <stddev>2e-4</stddev>
-                        <bias_mean>0.0000075</bias_mean>
-                        <bias_stddev>0.0000008</bias_stddev>
-                    </noise>
-                    </y>
-                    <z>
-                    <noise type="gaussian">
-                        <mean>0.0</mean>
-                        <stddev>2e-4</stddev>
-                        <bias_mean>0.0000075</bias_mean>
-                        <bias_stddev>0.0000008</bias_stddev>
-                    </noise>
-                    </z>
-                </angular_velocity>
-                <linear_acceleration>
-                    <x>
-                    <noise type="gaussian">
-                        <mean>0.0</mean>
-                        <stddev>1.7e-2</stddev>
-                        <bias_mean>0.1</bias_mean>
-                        <bias_stddev>0.001</bias_stddev>
-                    </noise>
-                    </x>
-                    <y>
-                    <noise type="gaussian">
-                        <mean>0.0</mean>
-                        <stddev>1.7e-2</stddev>
-                        <bias_mean>0.1</bias_mean>
-                        <bias_stddev>0.001</bias_stddev>
-                    </noise>
-                    </y>
-                    <z>
-                    <noise type="gaussian">
-                        <mean>0.0</mean>
-                        <stddev>1.7e-2</stddev>
-                        <bias_mean>0.1</bias_mean>
-                        <bias_stddev>0.001</bias_stddev>
-                    </noise>
-                    </z>
-                </linear_acceleration>
-                </imu> -->
-			</sensor>
-		</gazebo>
-	</xacro:macro>
+	  <!-- <gazebo reference="imu_link"> -->
+        <!-- <gravity>true</gravity> -->
+        <!-- <sensor name="imu_sensor" type="imu"> -->
+        <!-- <always_on>true</always_on> -->
+        <!-- <update_rate>100</update_rate> -->
+        <!-- <visualize>true</visualize> -->
+        <!-- <topic>__default_topic__</topic> -->
+        <!-- <plugin filename="libgazebo_ros_imu_sensor.so" name="imu_plugin"> -->
+            <!-- <topicName>imu</topicName> -->
+            <!-- <bodyName>imu_link</bodyName> -->
+            <!-- <updateRateHZ>10.0</updateRateHZ> -->
+            <!-- <gaussianNoise>0.0</gaussianNoise> -->
+            <!-- <xyzOffset>0 0 0</xyzOffset> -->
+            <!-- <rpyOffset>0 0 0</rpyOffset> -->
+            <!-- <frameName>imu_link</frameName> -->
+            <!-- <initialOrientationAsReference>false</initialOrientationAsReference> -->
+        <!-- </plugin> -->
+        <!-- <pose>0 0 0 0 0 0</pose> -->
+        <!-- </sensor> -->
+        <!-- </gazebo>	 -->
+</xacro:macro>
 </robot>

File: ribot_description/urdf/robot.urdf.xacro (robot description, xacro)
@@ -16,5 +16,5 @@
     <xacro:include filename="$(find ribot_description)/urdf/imu.urdf.xacro"/>
     <!-- Left IMU -->
-    <xacro:imu parent="tripod_left_support" prefix="imu" color_gazebo="Red">
+    <xacro:imu parent="left_support" prefix="imu" color_gazebo="Red">
         <origin xyz="0.015 0 0.02" rpy="0 0 0" />
         <color_rgb_rviz>
@@ -25,5 +25,5 @@
     </xacro:imu>
     <!-- Right Camera -->
-    <xacro:rgb_camera parent="tripod_right_support" prefix="rgb_right" color_gazebo="Green">
+    <xacro:rgb_camera parent="right_support" prefix="rgb_right" color_gazebo="Green">
         <origin xyz="0.015 0 0.012" rpy="0 0 0" />
         <color_rgb_rviz>
@@ -33,36 +33,5 @@
         </color_rgb_rviz>
     </xacro:rgb_camera>
-    <!-- Define links and joints -->
-    <link name="world" />
-    <!-- Tripod link-->
-    <link name="tripod">
-        <visual>
-            <origin xyz="0 0 0" rpy="0 0 0" />
-            <geometry>
-                <mesh filename="package://ribot_description/meshes/tripod/tripod.stl"
-                    scale="1 1 1" />
-            </geometry>
-            <material name="tripod_color" />
-        </visual>
-        <collision name="tripod_collision">
-            <origin xyz="0 0 0" rpy="0 0 0" />
-            <geometry>
-                <mesh filename="package://ribot_description/meshes/tripod/tripod.stl"
-                    scale="1 1 1" />
-            </geometry>
-        </collision>
-        <inertial>
-            <mass value="1.0" />
-            <origin xyz="0 0 0" rpy="0 0 0" />
-            <inertia ixx="1" ixy="0" ixz="0" iyy="1" iyz="0" izz="1" />
-        </inertial>
-    </link>
-    <!-- parent to tripod -->
-    <joint name="world_to_tripod" type="fixed">
-        <parent link="world" />
-        <child link="tripod" />
-        <origin xyz="0 0 0" rpy="0 0 0" />
-    </joint>
-    <link name="tripod_plate">
+    <link name="plate">
         <visual>
             <origin xyz="0 0 0" rpy="0 0 0" />
@@ -84,28 +53,18 @@
         </inertial>
     </link>
-    <!-- tripod to tripod plate-->
-    <joint name="tripod_to_tripod_plate" type="revolute">
-        <parent link="tripod" />
-        <child link="tripod_plate" />
-        <origin xyz=".01 .03 1.65" rpy="0 0.314 0" />
-        <!-- <calibration rising="0.0"/> -->
-        <!-- <dynamics damping="0.0" friction="0.0"/> -->
-        <limit effort="30" velocity="1.0" lower="-2.2" upper="0.7" />
-        <!-- <safety_controller k_velocity="10" k_position="15" soft_lower_limit="-2.0" soft_upper_limit="0.5" /> -->
-    </joint>
     <!-- Tripod left support-->
-    <link name="tripod_left_support" />
+    <link name="left_support" />
     <!-- tripod plate to tripod left support -->
-    <joint name="tripod_plate_to_tripod_left_support" type="fixed">
-        <parent link="tripod_plate" />
-        <child link="tripod_left_support" />
+    <joint name="plate_to_left_support" type="fixed">
+        <parent link="plate" />
+        <child link="left_support" />
         <origin xyz="0 0.18 0.0075" rpy="0 0 0" />
     </joint>
     <!-- Tripod right support-->
-    <link name="tripod_right_support" />
+    <link name="right_support" />
     <!-- tripod plate to tripod right support -->
-    <joint name="tripod_plate_to_tripod_right_support" type="fixed">
-        <parent link="tripod_plate" />
-        <child link="tripod_right_support" />
+    <joint name="plate_to_right_support" type="fixed">
+        <parent link="plate" />
+        <child link="right_support" />
         <origin xyz="0 -0.18 0.0075" rpy="0 0 0" />
     </joint>

Commit message: re-organized some files and readded the camera

File: ribot_description/urdf/imu.urdf.xacro (robot description, xacro)
@@ -1,5 +1,5 @@
 <?xml version="1.0"?>
 <robot name="imu" xmlns:xacro="http://ros.org/wiki/xacro">
-	<!-- This is a xacro macro to define and rgb camera.
+	<!-- This is a xacro macro to define an IMU.
 	You can define as arguments the parent coordinate frame, the name of the sensor, the transformation
 	from that parent frame to the camera's root frame, the color to be used in rviz, and the color
@@ -11,5 +11,5 @@
 	<xacro:macro name="imu" params="parent prefix *origin **color_rviz color_gazebo">
 		<joint name="${prefix}_joint" type="fixed">
-			<origin xyz="0.0 0.0 0.0" />
+			<xacro:insert_block name="origin"/>
 			<parent link="${parent}" />
 			<child link="${prefix}_link" />
@@ -36,25 +36,8 @@
 			</inertial>
 		</link>
-		<!-- IMU sensor-->
-	  <!-- <gazebo reference="imu_link"> -->
-        <!-- <gravity>true</gravity> -->
-        <!-- <sensor name="imu_sensor" type="imu"> -->
-        <!-- <always_on>true</always_on> -->
-        <!-- <update_rate>100</update_rate> -->
-        <!-- <visualize>true</visualize> -->
-        <!-- <topic>__default_topic__</topic> -->
-        <!-- <plugin filename="libgazebo_ros_imu_sensor.so" name="imu_plugin"> -->
-            <!-- <topicName>imu</topicName> -->
-            <!-- <bodyName>imu_link</bodyName> -->
-            <!-- <updateRateHZ>10.0</updateRateHZ> -->
-            <!-- <gaussianNoise>0.0</gaussianNoise> -->
-            <!-- <xyzOffset>0 0 0</xyzOffset> -->
-            <!-- <rpyOffset>0 0 0</rpyOffset> -->
-            <!-- <frameName>imu_link</frameName> -->
-            <!-- <initialOrientationAsReference>false</initialOrientationAsReference> -->
-        <!-- </plugin> -->
-        <!-- <pose>0 0 0 0 0 0</pose> -->
-        <!-- </sensor> -->
-        <!-- </gazebo>	 -->
+		<gazebo reference="${prefix}_link">
+			<selfCollide>false</selfCollide>
+			<material>Gazebo/${color_gazebo}</material>
+		</gazebo>
 </xacro:macro>
 </robot>

File: ribot_description/urdf/robot.urdf.xacro (robot description, xacro)
@@ -49,10 +49,29 @@
         </gazebo>
     </link>
-    <link name="imu">
-    </link>
-    <joint name="plate_to_imu" type="fixed">
+    <!-- <link name="imu">
+    </link> -->
+    <!-- <joint name="plate_to_imu" type="fixed">
       <origin xyz="0 0.1 -0.305" rpy="0 0 0"/>
       <parent link="plate"/>
       <child link="imu"/>
-    </joint>
+    </joint> -->
+    <!-- SENSORS -->
+    <!-- Left IMU -->
+    <xacro:imu parent="plate" prefix="imu" color_gazebo="Red">
+        <origin xyz="0.0 0.18 0.01" rpy="0 0 0" />
+        <color_rgb_rviz>
+            <material name="red">
+                <color rgba="0.9 0 0 1" />
+            </material>
+        </color_rgb_rviz>
+    </xacro:imu>
+    <!-- Right Camera -->
+    <xacro:rgb_camera parent="plate" prefix="rgb_right" color_gazebo="Green">
+        <origin xyz="0.015 -0.18 0.0195" rpy="0 0 0" />
+        <color_rgb_rviz>
+            <material name="green">
+                <color rgba="0 0.9 0 1" />
+            </material>
+        </color_rgb_rviz>
+    </xacro:rgb_camera>
 </robot>

Commit message: fix: added imu sensor plugin
now added an IMU sensor plugin that returns IMU sensor data, publishing
it in the topic /imu; for further

File: ribot_description/urdf/imu.urdf.xacro (robot description, xacro)
@@ -39,4 +39,20 @@
 			<selfCollide>false</selfCollide>
 			<material>Gazebo/${color_gazebo}</material>
+	    	<sensor name="imu_sensor" type="imu">
+				<always_on>true</always_on>
+				<update_rate>1000</update_rate>
+				<visualize>true</visualize>
+				<topic>/imu</topic>
+				<plugin filename="libgazebo_ros_imu_sensor.so" name="imu_plugin">
+					<topicName>/imu</topicName>
+					<bodyName>plate</bodyName>
+					<updateRateHZ>100.0</updateRateHZ>
+					<gaussianNoise>0.0</gaussianNoise>
+					<xyzOffset>0 0 0</xyzOffset>
+					<rpyOffset>0 0 0</rpyOffset>
+					<frameName>imu_link</frameName>
+					<initialOrientationAsReference>true</initialOrientationAsReference>
+				</plugin>
+			</sensor>
 		</gazebo>
 </xacro:macro>

File: ribot_description/urdf/robot.urdf.xacro (robot description, xacro)
@@ -21,12 +21,36 @@
     <xacro:include filename="$(find ribot_description)/urdf/rgb_camera.urdf.xacro" />
     <xacro:include filename="$(find ribot_description)/urdf/imu.urdf.xacro"/>
-    <!-- World link -->
-    <!-- <link name="world"/> -->
     <link name="base_link">
+        <xacro:default_inertial />
     </link>
-    <joint name="base_link_to_plate" type="fixed">
-      <origin xyz="0 0 0" rpy="0 0 0"/>
-      <parent link="base_link"/>
-      <child link="plate"/>
+    <joint name="base_link_to_prismatic_x" type="prismatic">
+        <origin xyz="0 0 0" rpy="0 0 0"/>
+        <parent link="base_link"/>
+        <child link="prismatic_x"/>
+        <axis xyz="1 0 0"/>
+        <limit effort="1000.0" lower="-0.38" upper="0" velocity="0.5"/>
+    </joint>
+    <link name="prismatic_x">
+        <visual>
+            <origin xyz="0 0 0" rpy="0 0 0" />
+            <geometry>
+                <box size="0.001 0.001 0.001" />
+            </geometry>
+        </visual>
+        <collision>
+            <origin xyz="0 0 0" rpy="0 0 0" />
+            <geometry>
+                <box size="0.001 0.001 0.001" />
+            </geometry>
+        </collision>
+        <xacro:default_inertial />
+        <gazebo>
+            <gravity>0</gravity>
+        </gazebo>
+    </link>
+    <joint name="prismatic_x_to_plate" type="fixed">
+        <parent link="prismatic_x"/>
+        <child link="plate"/>
+        <origin xyz="0.1 0 0" rpy="0 0 0"/>
     </joint>
     <link name="plate">
@@ -45,33 +69,40 @@
         </collision>
         <xacro:default_inertial />
-        <gazebo>
-            <gravity>0</gravity>
-        </gazebo>
     </link>
-    <!-- <link name="imu">
-    </link> -->
-    <!-- <joint name="plate_to_imu" type="fixed">
-      <origin xyz="0 0.1 -0.305" rpy="0 0 0"/>
-      <parent link="plate"/>
-      <child link="imu"/>
-    </joint> -->
+    <!-- GAZEBO -->
+    <!-- ROS control plugin -->
+    <gazebo>
+        <plugin name="gazebo_ros_control" filename="libgazebo_ros_control.so">
+            <namespace>/ribot</namespace>
+        </plugin>
+    </gazebo>
+    <!-- Transmissions -->
+    <transmission name="base_link_to_prismatic_x_trans">
+        <type>transmission_interfact/SimpleTransmission</type>
+        <actuator name="motor1">
+            <mechanicalReduction>1</mechanicalReduction>
+        </actuator>
+        <joint name="base_link_to_prismatic_x">
+            <hardwareInterface>hardware_interface/PositionJointInterface</hardwareInterface>
+        </joint>
+    </transmission>
     <!-- SENSORS -->
     <!-- Left IMU -->
-    <xacro:imu parent="plate" prefix="imu" color_gazebo="Red">
-        <origin xyz="0.0 0.18 0.01" rpy="0 0 0" />
-        <color_rgb_rviz>
-            <material name="red">
-                <color rgba="0.9 0 0 1" />
-            </material>
-        </color_rgb_rviz>
-    </xacro:imu>
+    <!-- <xacro:imu parent="plate" prefix="imu" color_gazebo="Red"> -->
+        <!-- <origin xyz="0.0 0.18 0.01" rpy="0 0 0" />           -->
+        <!-- <color_rgb_rviz> -->
+            <!-- <material name="red"> -->
+                <!-- <color rgba="0.9 0 0 1" /> -->
+            <!-- </material> -->
+        <!-- </color_rgb_rviz> -->
+    <!-- </xacro:imu> -->
     <!-- Right Camera -->
-    <xacro:rgb_camera parent="plate" prefix="rgb_right" color_gazebo="Green">
-        <origin xyz="0.015 -0.18 0.0195" rpy="0 0 0" />
-        <color_rgb_rviz>
-            <material name="green">
-                <color rgba="0 0.9 0 1" />
-            </material>
-        </color_rgb_rviz>
-    </xacro:rgb_camera>
+    <!-- <xacro:rgb_camera parent="plate" prefix="rgb_right" color_gazebo="Green"> -->
+        <!-- <origin xyz="0.015 -0.18 0.0195" rpy="0 0 0" /> -->
+        <!-- <color_rgb_rviz> -->
+            <!-- <material name="green"> -->
+                <!-- <color rgba="0 0.9 0 1" /> -->
+            <!-- </material> -->
+        <!-- </color_rgb_rviz> -->
+    <!-- </xacro:rgb_camera> -->
 </robot>

File: ribot_description/urdf/robot2.urdf.xacro (robot description, xacro)
@@ -17,4 +17,5 @@
         </inertial>
     </xacro:macro>
+    <xacro:include filename="$(find ribot_description)/urdf/imu.urdf.xacro"/>
     <!-- The Robot's base link -->
     <link name="base_link">
@@ -169,3 +170,13 @@
         </joint>
     </transmission>
+    <!-- SENSORS -->
+    <!-- Left IMU -->
+    <xacro:imu parent="plate" prefix="imu" color_gazebo="Red">
+        <origin xyz="0.0 0.18 0.01" rpy="0 0 0" />
+        <color_rgb_rviz>
+            <material name="red">
+                <color rgba="0.9 0 0 1" />
+            </material>
+        </color_rgb_rviz>
+    </xacro:imu>
 </robot>
